File: bicolour-matrix/bicolour-matrix.kicad_pcb (KiCad board)
At the start: 4 copper layers, 132.4 x 33.4 mm, 49 parts, among them J1 Conn_01x04_Pin, J2 Conn_01x04_Pin, J3 Conn_01x04_Socket, J4 Conn_01x04_Socket, J5 Conn_01x02_Socket, U1 HT16K33A-28SSOP, U2 HT16K33A-28SSOP, U3 HT16K33A-28SSOP, U4 HT16K33A-28SSOP

Commit message: feat: final update
Parts:
- added G***: LOGO, LOGO, B.Cu at (172.6, 88.0)
- added G***: LOGO, LOGO, B.Cu at (139.7, 87.3)
- moved JP5 1.84 mm to (130.0, 87.5)
- moved JP4 1.84 mm to (127.3, 87.5)
- moved JP6 1.84 mm to (132.6, 87.5)
- moved D2 1.83 mm to (130.0, 93.0)
- moved R3 1.80 mm to (128.7, 90.6)
- moved R4 1.80 mm to (129.9, 90.6)
- moved R5 1.80 mm to (131.2, 90.6)
- moved JP8 1.76 mm to (162.9, 87.5)
- moved JP7 1.76 mm to (160.3, 87.5)
- moved JP9 1.76 mm to (165.5, 87.5)
- moved D3 1.75 mm to (162.9, 93.0)
- moved R13 1.71 mm to (161.6, 90.6)
- moved R14 1.71 mm to (162.8, 90.6)
- moved R15 1.71 mm to (164.1, 90.6)
- moved JP10 1.69 mm to (193.2, 87.5)
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Routing:
- net /SDA: track 258.3 -> 254.5 mm
- net /Matrix 4/C7: track 15.4 -> 12.9 mm
- net /SCL: track 274.3 -> 271.9 mm
- net /Matrix 4/R2: track 40.0 -> 38.4 mm
- net /Matrix 2/R2: track 40.0 -> 38.4 mm
- net /Matrix 3/R2: track 40.0 -> 38.4 mm
- net /Matrix 3/R0: track 36.6 -> 35.1 mm
- net /Matrix 2/R0: track 36.6 -> 35.1 mm
- net /Matrix 4/R0: track 36.6 -> 35.1 mm
- net /Matrix 1/C0: track 22.7 -> 21.5 mm
- net /Matrix 1/R1: track 37.0 -> 38.1 mm
- net /Matrix 4/C5: track 16.6 -> 15.5 mm
- net /Matrix 2/R1: track 39.2 -> 38.1 mm
- net /Matrix 4/R1: track 39.2 -> 38.1 mm
- net /Matrix 3/R1: track 39.2 -> 38.1 mm
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Other:
- board text added: "SCL SDA"
- board text added: "matrix board v2"
- board text removed: "SCL"
- board text removed: "SDA"

Commit message: feat: better power connections
Routing:
- net GND: track 17.8 -> 9.09 mm, vias 10 -> 50
- net VDD: vias 11 -> 23
- added copper zone on F.Cu, net GND
