File: bicolour-matrix/bicolour-matrix.kicad_sch (KiCad schematic)
At the start: 4 parts, among them J1 Conn_01x04_Pin, J2 Conn_01x04_Pin

Commit message: feat: all changes
Parts:
- removed C1, C6: 10uF, PCM_JLCPCB:C_0805, symbol PCM_JLCPCB-Capacitors:0805,10uF
- added C1, C6: 10uF, PCM_JLCPCB:C_0805, symbol PCM_JLCPCB-Capacitors:0805,10uF,(2)
- added J3, J4: Conn_01x04_Socket, Connector_JST:JST_SH_SM04B-SRSS-TB_1x04-1MP_P1.00mm_Horizontal, symbol Connector:Conn_01x04_Socket
- added J5: Conn_01x02_Socket, Connector_PinSocket_2.54mm:PinSocket_1x02_P2.54mm_Vertical, symbol Connector:Conn_01x02_Socket
- added R1, R2: 10kΩ, Resistor_SMD:R_0603_1608Metric, symbol PCM_JLCPCB-Resistors:0603,10kΩ
Connections:
- net GND: now also C1.2, C6.2, J3.1 (Pin_1), J4.1 (Pin_1)
- net VDD: now also C1.1, C6.1, J3.2 (Pin_2), J4.2 (Pin_2), R1.1, R2.1
- net Matrix 1/SCL renamed SCL
- net SCL: now also J3.4 (Pin_4), J4.4 (Pin_4), J5.1 (Pin_1), R1.2
- net Matrix 1/SDA renamed SDA
- net SDA: now also J3.3 (Pin_3), J4.3 (Pin_3), J5.2 (Pin_2), R2.2
Other:
- moved on the sheet: J1, J2
