File: adapter-board-r2/adapter-board-r2.kicad_pcb (KiCad board)
At the start: 4 copper layers, 68.4 x 33.3 mm, 47 parts, among them J1 USB_C_Receptacle_USB2.0_14P, J2 Conn_01x02_Socket, J3 Conn_01x04_Socket, J4 Conn_01x07_Pin, Q1 UMH3N, Q2 BSS138W, Q3 BSS138W, U1 ESP32-C3-WROOM-02, U2 USBLC6-2SC6, U3 CH340X, U4 AP2114HA-3.3TRG1, U5 ENS210, U6 LIS2DW12TR, U7 SCD40-D-R2, U8 YSN8900AP3, U9 BMP580

Commit message: feat: updated pcb
Parts:
- added C18: 100nF, PCM_JLCPCB:C_0603, F.Cu at (120.1, 103.8)
- added R10: 0Ω, PCM_JLCPCB:R_0402, F.Cu at (103.8, 84.5)
- added R11: 0Ω, PCM_JLCPCB:R_0402, F.Cu at (106.6, 84.5)
- added R12: 0Ω, PCM_JLCPCB:R_0402, F.Cu at (107.5, 84.5)
- added R9: 0Ω, PCM_JLCPCB:R_0402, F.Cu at (104.7, 84.5)
- added U10: STCC4, custom:STCC4, F.Cu at (117.4, 103.9)
- U5: value ENS210 -> SHT4x; footprint Package_DFN_QFN:AMS_QFN-4-1EP_2x2mm_P0.95mm_EP0.7x1.6mm -> Sensor_Humidity:Sensirion_DFN-4_1.5x1.5mm_P0.8mm_SHT4x_NoCentralPad
- moved C12 16.3 mm to (134.2, 96.7)
- moved C13 16.3 mm to (133.7, 98.1)
- moved C14 16.3 mm to (133.1, 96.2)
- moved U6 16.3 mm to (135.9, 97.0)
- moved C16 9.23 mm to (98.7, 78.6)
- moved U9 9.23 mm to (98.7, 80.4)
- moved C15 9.23 mm to (96.6, 80.7)
- moved C8 5.95 mm to (105.9, 82.0), turned to 0 degrees
- moved U5 5.94 mm to (105.9, 80.2), turned to -90 degrees
- moved D1 1.07 mm to (101.8, 85.7), turned to 90 degrees
Connections:
- U5 pad 1: +3V3 -> Net-(U5-SDA)
- U5 pad 2: /SCL -> Net-(U5-SCL)
- U5 pad 3: /SDA -> +3V3
Routing:
- net /SCL_C: track 0.00 -> 25.1 mm, vias 0 -> 2
- net +5V: track 65.9 -> 90.3 mm, vias 5 -> 4
- net /SDA_C: track 0.00 -> 22.6 mm
- net /INT1: track 34.5 -> 16.8 mm
- net /SCK: track 31.9 -> 14.3 mm
- net /MISO: track 29.3 -> 11.8 mm
- net /MOSI: track 27.7 -> 10.1 mm
- net /SDA: track 126.7 -> 136.3 mm
- net /SCL: track 112.1 -> 119.1 mm, vias 5 -> 6
- net Net-(U5-SDA): track 0.00 -> 6.35 mm
- net Net-(U5-SCL): track 0.00 -> 6.24 mm
- net /CS_ACC: track 27.2 -> 22.3 mm
- net +3V3: track 32.9 -> 36.4 mm, vias 36 -> 37
- net Net-(U8-VBAT): track 3.16 -> 2.34 mm
- net /IO9: track 65.3 -> 65.9 mm
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Other:
- outline, holes or cut-outs redrawn

Commit message: feat: adapter, button changes
Parts:
- renumbered C8 to C10, C10 to C11, C17 to C12, C15 to C13, C16 to C14, C14 to C15, C12 to C16, C13 to C17, C7 to C3, C3 to C5, C5 to C6, C6 to C7, C9 to C8, C11 to C9, J4 to J2, J2 to J3, J3 to J4, R6 to R10, R7 to R11, R8 to R12, R9 to R5, R10 to R6, R11 to R7, R12 to R8, R5 to R9, U8 to U5, U5 to U6, U9 to U8, U6 to U9
Routing:
- net /PU: track 79.2 -> 78.9 mm, vias 4 -> 3
