File: adapter-board-r2/adapter-board-r2.kicad_pcb (KiCad board)
At the start: 4 copper layers, 68.4 x 33.3 mm, 53 parts, among them J1 USB_C_Receptacle_USB2.0_14P, J2 Conn_01x07_Pin, J3 Conn_01x02_Socket, J4 Conn_01x04_Socket, Q1 UMH3N, Q2 BSS138W, Q3 BSS138W, U1 ESP32-C3-WROOM-02, U10 STCC4, U2 USBLC6-2SC6, U3 CH340X, U4 AP2114HA-3.3TRG1, U5 YSN8900AP3, U6 SHT4x, U7 SCD40-D-R2, U8 BMP580, U9 LIS2DW12TR

Commit message: feat: final update
Parts:
- added G***: LOGO, LOGO, B.Cu at (118.8, 92.3)
Routing:
- net +5V: track 90.5 -> 91.2 mm
- net GND: vias 62 -> 86
Other:
- board text added: "5V 1A"
- board text added: "GND"
- board text added: "S1 S2 GND 3V3 SDA SCL INT"
- board text added: "SCL"
- board text added: "SDA"
- board text added: "adapter board v2"
