File: button-board-r2/button-board-r2.kicad_pcb (KiCad board)
At the start: 4 copper layers, 91.9 x 12.4 mm, 14 parts, among them J1 Conn_01x04_Socket, J2 Conn_01x07_Pin, J3 Conn_01x02_Pin, J4 Conn_01x02_Pin, U1 VEML6030, U2 TTP223-BA6-TD, U3 TTP223-BA6-TD

Commit message: feat: adapter, button changes
Parts:
- removed J3, J4: Conn_01x02_Pin, Connector_PinHeader_2.54mm:PinHeader_1x02_P2.54mm_Vertical
- J2: footprint Connector_PinHeader_2.54mm:PinHeader_1x07_P2.54mm_Vertical -> Connector_JST:JST_SH_SM07B-SRSS-TB_1x07-1MP_P1.00mm_Horizontal; moved to B.Cu
- moved J2 5.05 mm to (157.2, 106.9), turned to 180 degrees
Connections:
- J2 pad 1: /S2 -> /S1
- J2 pad 2: /S1 -> /S2
Routing:
- net /INT: track 36.3 -> 13.6 mm, vias 0 -> 1
- net /SCL: track 72.2 -> 53.3 mm
- net /SDA: track 68.6 -> 53.6 mm, vias 1 -> 3
- net /S1: track 17.0 -> 25.0 mm, vias 3 -> 0
- net /S2: track 13.6 -> 16.3 mm, vias 1 -> 0
- net GND: track 13.6 -> 14.8 mm, vias 7 -> 8
- net +3V3: track 6.79 -> 7.38 mm, vias 3 -> 4
