File: button-board-r2/button-board-r2.kicad_sch (KiCad schematic)
At the start: 14 parts, among them J1 Conn_01x04_Socket, J2 Conn_01x07_Pin, J3 Conn_01x02_Pin, J4 Conn_01x02_Pin, U1 VEML6030, U2 TTP223-BA6-TD, U3 TTP223-BA6-TD

Commit message: feat: adapter, button changes
Parts:
- removed J3, J4: Conn_01x02_Pin, Connector_PinHeader_2.54mm:PinHeader_1x02_P2.54mm_Vertical, symbol Connector:Conn_01x02_Pin
- J2: footprint Connector_PinHeader_2.54mm:PinHeader_1x07_P2.54mm_Vertical -> Connector_JST:JST_SH_SM07B-SRSS-TB_1x07-1MP_P1.00mm_Horizontal
Connections:
- net S1: now also J2.1 (Pin_1); no longer J2.2 (Pin_2)
- net S2: now also J2.2 (Pin_2); no longer J2.1 (Pin_1)
- no-connect marks 5 -> 1
Other:
- note added: "board connector"
- note removed: "board connectors"
- note removed: "mounting headers"
Changed lines of the file:
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@@
 	(generator_version "9.0")
 	(paper "A4")
-	(text "mounting headers"
-		(exclude_from_sim no)
-		(at 171.45 87.884 0)
-		(effects
-			(font
-				(size 1.27 1.27)
-			)
-		)
-	)
 	(text "touch sensors"
 		(exclude_from_sim no)
@@
 		)
 	)
-	(text "board connectors"
+	(text "board connector"
 		(exclude_from_sim no)
-		(at 155.194 97.028 0)
+		(at 137.668 94.234 0)
 		(effects
 			(font
@@
 	)
 	(no_connect
-		(at 173.99 83.82)
-	)
-	(no_connect
-		(at 173.99 73.66)
-	)
-	(no_connect
-		(at 173.99 71.12)
-	)
-	(no_connect
 		(at 109.22 128.27)
-	)
-	(no_connect
-		(at 173.99 81.28)
 	)
 	(wire
@@
 	)
 	(label "S2"
+		(at 134.62 73.66 0)
+		(effects
+			(font
+				(size 1.27 1.27)
+			)
+			(justify left bottom)
+		)
+	)
+	(label "S2"
 		(at 220.98 121.92 180)
 		(effects
@@
 		)
 	)
+	(label "S1"
+		(at 134.62 71.12 0)
+		(effects
+			(font
+				(size 1.27 1.27)
+			)
+			(justify left bottom)
+		)
+	)
 	(label "SCL"
 		(at 134.62 83.82 0)
@@
 	(label "INT"
 		(at 134.62 86.36 0)
-		(effects
-			(font
-				(size 1.27 1.27)
-			)
-			(justify left bottom)
-		)
-	)
-	(label "S2"
-		(at 134.62 71.12 0)
-		(effects
-			(font
-				(size 1.27 1.27)
-			)
-			(justify left bottom)
-		)
-	)
-	(label "S1"
-		(at 134.62 73.66 0)
 		(effects
 			(font
@@
 	)
 	(symbol
-		(lib_id "Connector:Conn_01x02_Pin")
-		(at 168.91 81.28 0)
-		(unit 1)
-		(exclude_from_sim no)
-		(in_bom yes)
-		(on_board yes)
-		(dnp no)
-		(fields_autoplaced yes)
-		(property "Reference" "J4"
-			(at 169.545 76.2 0)
-			(effects
-				(font
-					(size 1.27 1.27)
-				)
-			)
-		)
-		(property "Value" "Conn_01x02_Pin"
-			(at 169.545 78.74 0)
-			(effects
-				(font
-					(size 1.27 1.27)
-				)
-			)
-		)
-		(property "Footprint" "Connector_PinHeader_2.54mm:PinHeader_1x02_P2.54mm_Vertical"
-			(at 168.91 81.28 0)
-			(effects
-				(font
-					(size 1.27 1.27)
-				)
-				(hide yes)
-			)
-		)
-		(property "Datasheet" "~"
-			(at 168.91 81.28 0)
-			(effects
-				(font
-					(size 1.27 1.27)
-				)
-				(hide yes)
-			)
-		)
-		(property "Description" "Generic connector, single row, 01x02, script generated"
-			(at 168.91 81.28 0)
-			(effects
-				(font
-					(size 1.27 1.27)
-				)
-				(hide yes)
-			)
-		)
-		(pin "1"
-		)
-		(pin "2"
-		)
-		(instances
-			(project "button-board-r2"
-				(path "/c1054cca-9414-4084-a196-71cb409e4063"
-					(reference "J4")
-					(unit 1)
-				)
-			)
-		)
-	)
-	(symbol
 		(lib_id "Connector:Conn_01x04_Socket")
 		(at 57.15 121.92 0)
@@
 	)
 	(symbol
-		(lib_id "Connector:Conn_01x02_Pin")
-		(at 168.91 71.12 0)
-		(unit 1)
-		(exclude_from_sim no)
-		(in_bom yes)
-		(on_board yes)
-		(dnp no)
-		(fields_autoplaced yes)
-		(property "Reference" "J3"
-			(at 169.545 66.04 0)
-			(effects
-				(font
-					(size 1.27 1.27)
-				)
-			)
-		)
-		(property "Value" "Conn_01x02_Pin"
-			(at 169.545 68.58 0)
-			(effects
-				(font
-					(size 1.27 1.27)
-				)
-			)
-		)
-		(property "Footprint" "Connector_PinHeader_2.54mm:PinHeader_1x02_P2.54mm_Vertical"
-			(at 168.91 71.12 0)
-			(effects
-				(font
-					(size 1.27 1.27)
-				)
-				(hide yes)
-			)
-		)
-		(property "Datasheet" "~"
-			(at 168.91 71.12 0)
-			(effects
-				(font
-					(size 1.27 1.27)
-				)
-				(hide yes)
-			)
-		)
-		(property "Description" "Generic connector, single row, 01x02, script generated"
-			(at 168.91 71.12 0)
-			(effects
-				(font
-					(size 1.27 1.27)
-				)
-				(hide yes)
-			)
-		)
-		(pin "1"
-		)
-		(pin "2"
-		)
-		(instances
-			(project "button-board-r2"
-				(path "/c1054cca-9414-4084-a196-71cb409e4063"
-					(reference "J3")
-					(unit 1)
-				)
-			)
-		)
-	)
-	(symbol
 		(lib_id "PCM_JLCPCB-Capacitors:0603,22pF")
 		(at 220.98 133.35 0)
@@
 			)
 		)
-		(property "Footprint" "Connector_PinHeader_2.54mm:PinHeader_1x07_P2.54mm_Vertical"
+		(property "Footprint" "Connector_JST:JST_SH_SM07B-SRSS-TB_1x07-1MP_P1.00mm_Horizontal"
 			(at 128.27 78.74 0)
 			(effects
